File: Harsch_Systems_RP2040_SMD.sch (KiCad schematic (older format))
At the start: 32 parts, among them J1 Jack-DC, J2 USB_A, J3 DEBUG, J4 Conn_01x08_Female, J5 Conn_01x08_Female, J6 Conn_01x04_Female, J7 Conn_01x06_Female, SW1 SW_MEC_5E, U1 RP2040, U2 W25Q32JVSSIQ_TR, Y1 12MHz

Commit message: Updates, cleanup, and component association.
Connections:
- net labels added: +10V, +24V, ADC0, ADC1, ADC2, ADC3, GPIO1, GPIO11, GPIO13, GPIO15, GPIO3, GPIO5, GPIO7, GPIO9, PWM0, PWM1, PWM2, PWM3, PWM4, PWM5, PWM6, PWM7
- net labels removed: USB_BOOT
- wire segments 192 -> 248
- no-connect marks 0 -> 11
Other:
- note added: "12 MHz CLOCK"
- note added: "DEBUG PORT"
- note added: "DECOUPLING CAPACITORS"
- note added: "FLASH MEMORY"
- note added: "INPUTS + OUTPUTS"
- note added: "RP2040"
- note added: "USB"
- moved on the sheet: C1, C10, C11, C12, C13, C14, C2, C3, C4, C5, C6, C7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

Commit message: Finished the schematic, except for maybe a couple test points.
Parts:
- added C1, C5: 1μ, Capacitor_SMD:C_0805_2012Metric, symbol Device:C
- added C12, C16: 22μ, Capacitor_SMD:C_0805_2012Metric, symbol Device:C
- added C14, C2: 0.1μ, Capacitor_SMD:C_0603_1608Metric, symbol Device:C
- added C3, C8: 33n, Capacitor_SMD:C_0805_2012Metric, symbol Device:C
- added C4: 10μ, Capacitor_SMD:C_0805_2012Metric, symbol Device:C
- added D1: LED, symbol Device:LED
- added D2: D_Schottky, Diode_SMD:D_SOD-123, symbol Device:D_Schottky
- added J2: Conn_01x02_Male, Connector_PinSocket_2.54mm:PinSocket_1x02_P2.54mm_Vertical, symbol Connector:Conn_01x02_Male
- added L1: 6.8μ, Inductor_SMD:L_Vishay_IHLP-2020, symbol Device:L_Core_Iron
- added R1: 10K, Resistor_SMD:R_0805_2012Metric, symbol Device:R_US
- added R3: 10k, Resistor_SMD:R_0805_2012Metric, symbol Device:R_US
- added R4: 53.6k, Resistor_SMD:R_0805_2012Metric, symbol Device:R_US
- added R81: 470, symbol Device:R_US
- added U1: XC6210B332MR, Package_TO_SOT_SMD:SOT-23-5, symbol Regulator_Linear:XC6210B332MR
- added U2: TPS62933, Package_DFN_QFN:Texas_VSON-HR-8_1.5x2mm_P0.5mm, symbol Custom_Parts:TPS62933
- R7: renamed from R6; value R_US -> DNP
- SW1: footprint Button_Switch_SMD:Panasonic_EVQPUJ_EVQPUA -> Button_Switch_SMD:SW_SPST_Omron_B3FS-100xP
- renumbered C4 to C10, C5 to C11, C6 to C13, C7 to C15, C8 to C17, C9 to C18, C10 to C19, C11 to C20, C12 to C21, C13 to C22, C14 to C23, C1 to C6, C2 to C7, C3 to C9, J4 to J3, J5 to J4, J6 to J5, J7 to J6, J2 to J7, J3 to J8, R7 to R10, R3 to R2, R4 to R5, R5 to R6, R1 to R8, R2 to R9, U1 to U3, U2 to U4
Connections:
- net labels added: +5V, GPIO25
- net labels removed: +10V
- wire segments 248 -> 304
Other:
- note added: "24V to 5V DC/DC Converter"
- note added: "5V to 3.3V Linear Voltage Regulator"
- note added: "LED"
- note added: "Power Flag Labels"
- moved on the sheet: J1

Commit message: Starting routing
Parts:
- added TP1, TP2, TP3, TP4: TestPoint, Connector_PinSocket_2.54mm:PinSocket_1x01_P2.54mm_Vertical, symbol Connector:TestPoint
- C10, C11, C13, C15, C17, C6, C7, C9: footprint Capacitor_SMD:C_0603_1608Metric -> Capacitor_SMD:C_0402_1005Metric_Pad0.74x0.62mm_HandSolder
- D1: footprint (none) -> LED_SMD:LED_0805_2012Metric
- R81: footprint (none) -> Resistor_SMD:R_0805_2012Metric
Changed lines of the file:
@@
 F 0 "C9" H 4665 1046 50  0000 L CNN
 F 1 "0.1μ" H 4665 955 50  0000 L CNN
-F 2 "Capacitor_SMD:C_0603_1608Metric" H 4588 850 50  0001 C CNN
+F 2 "Capacitor_SMD:C_0402_1005Metric_Pad0.74x0.62mm_HandSolder" H 4588 850 50  0001 C CNN
 F 3 "~" H 4550 1000 50  0001 C CNN
 	1    4550 1000
@@
 F 0 "C10" H 5065 1046 50  0000 L CNN
 F 1 "0.1μ" H 5065 955 50  0000 L CNN
-F 2 "Capacitor_SMD:C_0603_1608Metric" H 4988 850 50  0001 C CNN
+F 2 "Capacitor_SMD:C_0402_1005Metric_Pad0.74x0.62mm_HandSolder" H 4988 850 50  0001 C CNN
 F 3 "~" H 4950 1000 50  0001 C CNN
 	1    4950 1000
@@
 F 0 "C11" H 5465 1046 50  0000 L CNN
 F 1 "0.1μ" H 5465 955 50  0000 L CNN
-F 2 "Capacitor_SMD:C_0603_1608Metric" H 5388 850 50  0001 C CNN
+F 2 "Capacitor_SMD:C_0402_1005Metric_Pad0.74x0.62mm_HandSolder" H 5388 850 50  0001 C CNN
 F 3 "~" H 5350 1000 50  0001 C CNN
 	1    5350 1000
@@
 F 0 "C13" H 5865 1046 50  0000 L CNN
 F 1 "0.1μ" H 5865 955 50  0000 L CNN
-F 2 "Capacitor_SMD:C_0603_1608Metric" H 5788 850 50  0001 C CNN
+F 2 "Capacitor_SMD:C_0402_1005Metric_Pad0.74x0.62mm_HandSolder" H 5788 850 50  0001 C CNN
 F 3 "~" H 5750 1000 50  0001 C CNN
 	1    5750 1000
@@
 F 0 "C15" H 6265 1046 50  0000 L CNN
 F 1 "0.1μ" H 6265 955 50  0000 L CNN
-F 2 "Capacitor_SMD:C_0603_1608Metric" H 6188 850 50  0001 C CNN
+F 2 "Capacitor_SMD:C_0402_1005Metric_Pad0.74x0.62mm_HandSolder" H 6188 850 50  0001 C CNN
 F 3 "~" H 6150 1000 50  0001 C CNN
 	1    6150 1000
@@
 F 0 "C17" H 6665 1046 50  0000 L CNN
 F 1 "0.1μ" H 6665 955 50  0000 L CNN
-F 2 "Capacitor_SMD:C_0603_1608Metric" H 6588 850 50  0001 C CNN
+F 2 "Capacitor_SMD:C_0402_1005Metric_Pad0.74x0.62mm_HandSolder" H 6588 850 50  0001 C CNN
 F 3 "~" H 6550 1000 50  0001 C CNN
 	1    6550 1000
@@
 Wire Wire Line
 	3600 5400 3900 5400
-$Comp
-L power:+3.3V #PWR016
-U 1 1 60FE13F9
-P 4350 1950
-F 0 "#PWR016" H 4350 1800 50  0001 C CNN
-F 1 "+3.3V" H 4365 2123 50  0000 C CNN
-F 2 "" H 4350 1950 50  0001 C CNN
-F 3 "" H 4350 1950 50  0001 C CNN
-	1    4350 1950
-	1    0    0    -1
-$EndComp
 Wire Wire Line
 	4350 2050 4350 1950
@@
 Wire Wire Line
 	4450 1950 4350 1950
-Connection ~ 4350 1950
 $Comp
 L power:+3.3V #PWR017
@@
 F 0 "C6" H 3865 1046 50  0000 L CNN
 F 1 "0.1μ" H 3865 955 50  0000 L CNN
-F 2 "Capacitor_SMD:C_0603_1608Metric" H 3788 850 50  0001 C CNN
+F 2 "Capacitor_SMD:C_0402_1005Metric_Pad0.74x0.62mm_HandSolder" H 3788 850 50  0001 C CNN
 F 3 "~" H 3750 1000 50  0001 C CNN
 	1    3750 1000
@@
 F 0 "C7" H 4265 1046 50  0000 L CNN
 F 1 "0.1μ" H 4265 955 50  0000 L CNN
-F 2 "Capacitor_SMD:C_0603_1608Metric" H 4188 850 50  0001 C CNN
+F 2 "Capacitor_SMD:C_0402_1005Metric_Pad0.74x0.62mm_HandSolder" H 4188 850 50  0001 C CNN
 F 3 "~" H 4150 1000 50  0001 C CNN
 	1    4150 1000
@@
 F 0 "D1" H 2143 2845 50  0000 C CNN
 F 1 "LED" H 2143 2936 50  0000 C CNN
-F 2 "" H 2150 3100 50  0001 C CNN
+F 2 "LED_SMD:LED_0805_2012Metric" H 2150 3100 50  0001 C CNN
 F 3 "~" H 2150 3100 50  0001 C CNN
 	1    2150 3100
@@
 F 0 "R81" V 1445 3100 50  0000 C CNN
 F 1 "470" V 1536 3100 50  0000 C CNN
-F 2 "" V 1690 3090 50  0001 C CNN
+F 2 "Resistor_SMD:R_0805_2012Metric" V 1690 3090 50  0001 C CNN
 F 3 "~" H 1650 3100 50  0001 C CNN
 	1    1650 3100
@@
 Wire Notes Line
 	500  500  500  3350
-Text Notes 1850 3300 0    50   ~ 0
+Text Notes 1800 3300 0    50   ~ 0
 LED
+$Comp
+L Connector:TestPoint TP4
+U 1 1 6201CA69
+P 6500 6800
+F 0 "TP4" H 6558 6918 50  0000 L CNN
+F 1 "TestPoint" H 6558 6827 50  0000 L CNN
+F 2 "Connector_PinSocket_2.54mm:PinSocket_1x01_P2.54mm_Vertical" H 6700 6800 50  0001 C CNN
+F 3 "~" H 6700 6800 50  0001 C CNN
+	1    6500 6800
+	1    0    0    -1
+$EndComp
+$Comp
+L Connector:TestPoint TP1
+U 1 1 6201D638
+P 2550 6800
+F 0 "TP1" H 2608 6918 50  0000 L CNN
+F 1 "TestPoint" H 2608 6827 50  0000 L CNN
+F 2 "Connector_PinSocket_2.54mm:PinSocket_1x01_P2.54mm_Vertical" H 2750 6800 50  0001 C CNN
+F 3 "~" H 2750 6800 50  0001 C CNN
+	1    2550 6800
+	1    0    0    -1
+$EndComp
+$Comp
+L Connector:TestPoint TP3
+U 1 1 6201DEEB
+P 3000 1900
+F 0 "TP3" V 2954 2088 50  0000 L CNN
+F 1 "TestPoint" V 3045 2088 50  0000 L CNN
+F 2 "Connector_PinSocket_2.54mm:PinSocket_1x01_P2.54mm_Vertical" H 3200 1900 50  0001 C CNN
+F 3 "~" H 3200 1900 50  0001 C CNN
+	1    3000 1900
+	0    1    1    0
+$EndComp
+Connection ~ 3000 1900
+$Comp
+L Connector:TestPoint TP2
+U 1 1 6201F89F
+P 2650 900
+F 0 "TP2" V 2604 1088 50  0000 L CNN
+F 1 "TestPoint" V 2695 1088 50  0000 L CNN
+F 2 "Connector_PinSocket_2.54mm:PinSocket_1x01_P2.54mm_Vertical" H 2850 900 50  0001 C CNN
+F 3 "~" H 2850 900 50  0001 C CNN
+	1    2650 900
+	0    1    1    0
+$EndComp
+Connection ~ 2650 900
+$Comp
+L power:+1V1 #PWR016
+U 1 1 6208784A
+P 4350 1950
+F 0 "#PWR016" H 4350 1800 50  0001 C CNN
+F 1 "+1V1" H 4365 2123 50  0000 C CNN
+F 2 "" H 4350 1950 50  0001 C CNN
+F 3 "" H 4350 1950 50  0001 C CNN
+	1    4350 1950
+	1    0    0    -1
+$EndComp
+Connection ~ 4350 1950
 $EndSCHEMATC

Commit message: Power circuitry routing and board outline
Parts:
- removed C1: 1μ, Capacitor_SMD:C_0805_2012Metric, symbol Device:C
- removed C3: 33n, Capacitor_SMD:C_0805_2012Metric, symbol Device:C
- removed J2: Conn_01x02_Male, Connector_PinSocket_2.54mm:PinSocket_1x02_P2.54mm_Vertical, symbol Connector:Conn_01x02_Male
- removed U2: TPS62933, Package_DFN_QFN:Texas_VSON-HR-8_1.5x2mm_P0.5mm, symbol Custom_Parts:TPS62933
- added R82: 10, Resistor_SMD:R_0805_2012Metric, symbol Device:R_US
- added U11: TPS56339DDC, Package_TO_SOT_SMD:SOT-23-6, symbol Regulator_Switching:TPS56339DDC
- C8: value 33n -> .1μ
- L1: value 6.8μ -> 5.6μ
- R4: value 53.6k -> 52.3k
Connections:
- wire segments 304 -> 297
Other:
- moved on the sheet: C12, C14, C16, C8, L1, R3
